File: Atari TTP and OS.kicad_pcb (KiCad board)
At the start: 2 copper layers, 19.6 x 52.1 mm, 13 parts, among them J1 Left, J2 Right, J4 Signals, J6 TTP_sel, U1 74LS157, U2 27C010, U3 74LVC2G74

Commit message: Tracking
Routing:
- net GND: track 34.0 -> 85.1 mm, vias 0 -> 16
- net PB2: track 0.00 -> 41.0 mm, vias 0 -> 1
- net PB3: track 0.25 -> 34.5 mm, vias 0 -> 1
- net Net-(U1-Pad7): track 0.00 -> 27.4 mm, vias 0 -> 2
- net A16: track 0.00 -> 24.1 mm, vias 0 -> 2
- net VCC: track 69.4 -> 82.3 mm
- net Net-(J6-Pad1): track 0.00 -> 11.4 mm
- net Net-(D1-Pad1): track 13.4 -> 19.2 mm
- net Net-(C1-Pad1): track 16.5 -> 20.8 mm
- net D3: track 15.6 -> 11.7 mm
- net RST: track 0.63 -> 4.54 mm
- net A9: track 17.3 -> 15.5 mm
- net A11: track 23.6 -> 23.1 mm
- added copper zone on B.Cu, net GND
- added copper zone on F.Cu, net GND

Commit message: origin master
Other:
- board text added: "74LS157"
Changed lines of the file:
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@@
   (general
     (thickness 1.6)
-    (drawings 16)
+    (drawings 17)
     (tracks 357)
     (zones 0)
@@
   )
   (setup
-    (last_trace_width 0.508)
+    (last_trace_width 0.25)
     (user_trace_width 0.254)
     (user_trace_width 0.3048)
@@
     (solder_mask_min_width 0.25)
     (aux_axis_origin 122.428 104.902)
-    (visible_elements 7FFFFFFF)
+    (visible_elements 7FFFEFFF)
     (pcbplotparams
       (layerselection 0x010f0_ffffffff)
@@
     (tags "resistor handsolder")
     (attr smd)
-    (fp_text reference R3 (at 0 -1.82 90) (layer F.SilkS)
+    (fp_text reference R3 (at -3.2004 -0.0635 180) (layer F.SilkS)
       (effects (font (size 1 1) (thickness 0.15)))
     )
@@
     (descr "Through hole straight pin header, 1x02, 2.54mm pitch, single row")
     (tags "Through hole pin header THT 1x02 2.54mm single row")
-    (fp_text reference J6 (at 0 -2.33 90) (layer F.SilkS)
+    (fp_text reference J6 (at -0.635 -2.1844 90) (layer F.SilkS)
       (effects (font (size 1 1) (thickness 0.15)))
     )
@@
     (tags "resistor handsolder")
     (attr smd)
-    (fp_text reference R2 (at -3.2004 0.0508) (layer F.SilkS)
+    (fp_text reference R2 (at 3.2512 0.0381) (layer F.SilkS)
       (effects (font (size 1 1) (thickness 0.15)))
     )
@@
     (tags "resistor handsolder")
     (attr smd)
-    (fp_text reference R1 (at -3.0988 0.0762 90) (layer F.SilkS)
+    (fp_text reference R1 (at -0.6223 4.4704 90) (layer F.SilkS)
       (effects (font (size 1 1) (thickness 0.15)))
     )
@@
     (tags "diode handsolder")
     (attr smd)
-    (fp_text reference D2 (at 3.048 0.0762 270) (layer F.SilkS)
+    (fp_text reference D2 (at 2.0955 -2.1082 270) (layer F.SilkS)
       (effects (font (size 1 1) (thickness 0.15)))
     )
@@
     (tags "diode handsolder")
     (attr smd)
-    (fp_text reference D1 (at 3.1242 0.2032 270) (layer F.SilkS)
+    (fp_text reference D1 (at -3.4163 0.2794 270) (layer F.SilkS)
       (effects (font (size 1 1) (thickness 0.15)))
     )
@@
     )
   )
+  (gr_text 74LS157 (at 133.2484 77.1144 90) (layer F.SilkS)
+    (effects (font (size 1 1) (thickness 0.15)))
+  )
   (gr_text TTP (at 125.6792 54.0766) (layer F.SilkS)
     (effects (font (size 1 1) (thickness 0.15)))
@@
   (gr_line (start 141.986 52.832) (end 141.986 104.902) (layer Edge.Cuts) (width 0.05))
   (gr_line (start 122.428 52.832) (end 141.986 52.832) (layer Edge.Cuts) (width 0.05))
-  (gr_text PB2 (at 137.2616 54.9656 90) (layer F.SilkS)
-    (effects (font (size 0.8 0.8) (thickness 0.12)))
-  )
-  (gr_text PB3 (at 134.7216 55.0164 90) (layer F.SilkS)
-    (effects (font (size 0.8 0.8) (thickness 0.12)))
+  (gr_text PB2 (at 137.3378 54.737 90) (layer F.SilkS)
+    (effects (font (size 1 1) (thickness 0.15)))
+  )
+  (gr_text PB3 (at 134.7216 54.7624 90) (layer F.SilkS)
+    (effects (font (size 1 1) (thickness 0.15)))
   )
   (gr_text D6XX (at 132.1562 54.6354 90) (layer F.SilkS)
     (effects (font (size 0.8 0.8) (thickness 0.12)))
   )
-  (gr_text Rst (at 129.667 55.245 90) (layer F.SilkS)
-    (effects (font (size 0.8 0.8) (thickness 0.12)))
+  (gr_text Rst (at 129.6924 55.0164 90) (layer F.SilkS)
+    (effects (font (size 1 1) (thickness 0.15)))
   )
   (gr_line (start 125.7808 55.0418) (end 125.7808 55.3466) (layer F.SilkS) (width 0.12))
@@
     (effects (font (size 1 1) (thickness 0.15)))
   )
-  (via (at 131.064 93.726) (size 0.9) (drill 0.5) (layers F.Cu B.Cu) (net 2))
-  (via (at 131.064 96.52) (size 0.9) (drill 0.5) (layers F.Cu B.Cu) (net 2))
-  (via (at 133.35 96.52) (size 0.9) (drill 0.5) (layers F.Cu B.Cu) (net 2))
   (segment (start 124.910799 64.103199) (end 124.5108 63.7032) (width 0.6096) (layer B.Cu) (net 1))
   (segment (start 123.6628 61.6294) (end 123.6628 62.8552) (width 0.4064) (layer F.Cu) (net 1))
@@
   (segment (start 137.3124 81.915) (end 137.3124 81.1784) (width 0.6096) (layer F.Cu) (net 1))
   (segment (start 137.3124 81.1784) (end 137.7442 80.7466) (width 0.6096) (layer F.Cu) (net 1))
+  (via (at 131.064 93.726) (size 0.9) (drill 0.5) (layers F.Cu B.Cu) (net 2))
+  (via (at 131.064 96.52) (size 0.9) (drill 0.5) (layers F.Cu B.Cu) (net 2))
+  (via (at 133.35 96.52) (size 0.9) (drill 0.5) (layers F.Cu B.Cu) (net 2))
   (segment (start 130.9878 102.4128) (end 130.9878 101.6254) (width 0.8128) (layer F.Cu) (net 2))
   (segment (start 129.794001 103.606599) (end 130.9878 102.4128) (width 0.8128) (layer F.Cu) (net 2))
@@
   (segment (start 128.4478 88.4682) (end 125.857 85.8774) (width 0.3048) (layer B.Cu) (net 21))
   (segment (start 138.0236 97.8154) (end 139.8778 97.8154) (width 0.3048) (layer B.Cu) (net 22))
-  (segment (start 137.3378 98.5012) (end 138.0236 97.8154) (width 0.3048) (layer B.Cu) (net 22))
-  (segment (start 137.3378 99.7458) (end 137.3378 98.5012) (width 0.3048) (layer B.Cu) (net 22))
-  (segment (start 136.7282 100.3554) (end 137.3378 99.7458) (width 0.3048) (layer B.Cu) (net 22))
+  (segment (start 137.3632 98.4758) (end 138.0236 97.8154) (width 0.3048) (layer B.Cu) (net 22))
+  (segment (start 137.3632 99.7204) (end 137.3632 98.4758) (width 0.3048) (layer B.Cu) (net 22))
+  (segment (start 136.7282 100.3554) (end 137.3632 99.7204) (width 0.3048) (layer B.Cu) (net 22))
   (segment (start 133.5278 99.0854) (end 134.7978 100.3554) (width 0.3048) (layer B.Cu) (net 22))
   (segment (start 134.7978 100.3554) (end 136.7282 100.3554) (width 0.3048) (layer B.Cu) (net 22))
@@
   (segment (start 128.4478 86.3854) (end 126.4412 84.3788) (width 0.3048) (layer B.Cu) (net 25))
   (segment (start 126.4412 84.3788) (end 126.4412 74.2188) (width 0.3048) (layer B.Cu) (net 25))
-  (segment (start 132.1816 100.2792) (end 130.9878 99.0854) (width 0.3048) (layer F.Cu) (net 26))
+  (segment (start 132.2578 100.3554) (end 130.9878 99.0854) (width 0.3048) (layer F.Cu) (net 26))
   (segment (start 139.6238 103.1494) (end 135.4582 103.1494) (width 0.3048) (layer F.Cu) (net 26))
   (segment (start 139.8778 102.8954) (end 139.6238 103.1494) (width 0.3048) (layer F.Cu) (net 26))
   (segment (start 135.4582 103.1494) (end 134.7978 102.489) (width 0.3048) (layer F.Cu) (net 26))
   (segment (start 134.7978 102.489) (end 134.7978 100.7618) (width 0.3048) (layer F.Cu) (net 26))
-  (segment (start 134.7978 100.7618) (end 134.3152 100.2792) (width 0.3048) (layer F.Cu) (net 26))
-  (segment (start 134.3152 100.2792) (end 132.1816 100.2792) (width 0.3048) (layer F.Cu) (net 26))
+  (segment (start 134.7978 100.7618) (end 134.3914 100.3554) (width 0.3048) (layer F.Cu) (net 26))
+  (segment (start 134.3914 100.3554) (end 132.2578 100.3554) (width 0.3048) (layer F.Cu) (net 26))
   (via (at 125.6284 60.0964) (size 0.9) (drill 0.5) (layers F.Cu B.Cu) (net 27))
   (segment (start 125.6128 61.6294) (end 125.6128 60.112) (width 0.3048) (layer F.Cu) (net 27))
